File: Eagle/PSoC_PyunPyun_Mini.brd (EAGLE design)
At the start: 57.1 x 52.1 mm, 28 parts, among them IC1 NJM2732

Commit message: シールドの製作完了
Routing:
- net SDA: track 22.9 -> 27.9 mm
- net SCL: track 27.9 -> 33.0 mm
Other:
- board size 57.1 x 52.1 mm -> 59.7 x 52.1 mm
Changed lines of the file:
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@@
 <layer number="97" name="Info" color="7" fill="1" visible="no" active="no"/>
 <layer number="98" name="Guide" color="6" fill="1" visible="no" active="no"/>
-<layer number="100" name="Grid" color="7" fill="1" visible="no" active="yes"/>
+<layer number="100" name="Grid" color="7" fill="1" visible="yes" active="yes"/>
 </layers>
 <board>
 <plain>
-<wire x1="56.82" y1="0" x2="56.82" y2="52.06" width="0" layer="20"/>
-<wire x1="56.82" y1="52.06" x2="0" y2="52.06" width="0" layer="20"/>
+<wire x1="59.36" y1="0" x2="59.36" y2="52.06" width="0" layer="20"/>
+<wire x1="59.36" y1="52.06" x2="0" y2="52.06" width="0" layer="20"/>
 <wire x1="0" y1="52.06" x2="0" y2="43.18" width="0" layer="20"/>
 <wire x1="0" y1="15.24" x2="0" y2="0" width="0" layer="20"/>
@@
 <wire x1="0" y1="43.18" x2="2.54" y2="45.72" width="0.4064" layer="20"/>
 <wire x1="2.54" y1="45.72" x2="2.54" y2="52.07" width="0.4064" layer="20"/>
-<wire x1="2.54" y1="52.07" x2="57.15" y2="52.07" width="0.4064" layer="20"/>
-<wire x1="57.15" y1="52.07" x2="57.15" y2="1.27" width="0.4064" layer="20"/>
-<wire x1="57.15" y1="1.27" x2="2.54" y2="1.27" width="0.4064" layer="20"/>
+<wire x1="2.54" y1="52.07" x2="59.69" y2="52.07" width="0.4064" layer="20"/>
+<wire x1="59.69" y1="52.07" x2="59.69" y2="1.27" width="0.4064" layer="20"/>
+<wire x1="59.69" y1="1.27" x2="2.54" y2="1.27" width="0.4064" layer="20"/>
 <wire x1="2.54" y1="1.27" x2="2.54" y2="12.7" width="0.4064" layer="20"/>
 <wire x1="2.54" y1="12.7" x2="0" y2="15.24" width="0.4064" layer="20"/>
@@
 <wire x1="58.42" y1="7.62" x2="-2.54" y2="7.62" width="0" layer="100"/>
 <wire x1="-2.54" y1="5.08" x2="58.42" y2="5.08" width="0.254" layer="100" style="shortdash"/>
-<wire x1="0" y1="0" x2="57.15" y2="0" width="0" layer="20"/>
+<wire x1="0" y1="0" x2="59.36" y2="0" width="0" layer="20"/>
 <rectangle x1="3.81" y1="44.45" x2="41.91" y2="46.99" layer="39"/>
 <rectangle x1="3.81" y1="6.35" x2="54.61" y2="8.89" layer="39"/>
 <rectangle x1="41.91" y1="46.99" x2="44.45" y2="49.53" layer="39"/>
+<wire x1="59.36" y1="0" x2="59.69" y2="0" width="0" layer="20"/>
+<wire x1="55.88" y1="53.34" x2="55.88" y2="0" width="0" layer="100"/>
+<wire x1="58.42" y1="0" x2="58.42" y2="53.34" width="0" layer="100"/>
 </plain>
 <attributes>
@@
 <contactref element="JP4" pad="4"/>
 <contactref element="JP4" pad="8"/>
-<wire x1="50.8" y1="33.02" x2="43.18" y2="33.02" width="0.4064" layer="16"/>
-<wire x1="43.18" y1="33.02" x2="43.18" y2="22.86" width="0.4064" layer="16"/>
-<wire x1="43.18" y1="22.86" x2="40.64" y2="22.86" width="0.4064" layer="16"/>
+<wire x1="50.8" y1="33.02" x2="45.72" y2="33.02" width="0.4064" layer="16"/>
+<wire x1="45.72" y1="33.02" x2="45.72" y2="22.86" width="0.4064" layer="16"/>
+<wire x1="45.72" y1="22.86" x2="40.64" y2="22.86" width="0.4064" layer="16"/>
 <wire x1="50.8" y1="22.86" x2="54.61" y2="22.86" width="0.4064" layer="1"/>
 <wire x1="54.61" y1="22.86" x2="54.61" y2="33.02" width="0.4064" layer="1"/>
@@
 <signal name="RST">
 <contactref element="JP4" pad="7"/>
-<wire x1="45.72" y1="20.32" x2="45.72" y2="30.48" width="0.4064" layer="16"/>
-<wire x1="45.72" y1="30.48" x2="50.8" y2="30.48" width="0.4064" layer="16"/>
+<wire x1="48.26" y1="20.32" x2="48.26" y2="30.48" width="0.4064" layer="16"/>
+<wire x1="48.26" y1="30.48" x2="50.8" y2="30.48" width="0.4064" layer="16"/>
 <contactref element="R6" pad="2"/>
 <contactref element="R7" pad="2"/>
-<wire x1="43.18" y1="20.32" x2="45.72" y2="20.32" width="0.4064" layer="16"/>
+<wire x1="43.18" y1="20.32" x2="48.26" y2="20.32" width="0.4064" layer="16"/>
 <wire x1="40.64" y1="12.7" x2="40.64" y2="17.78" width="0.4064" layer="16"/>
 <wire x1="40.64" y1="17.78" x2="43.18" y2="17.78" width="0.4064" layer="16"/>
@@
 <contactref element="JP3" pad="1"/>
 <contactref element="JP4" pad="6"/>
-<wire x1="53.34" y1="5.08" x2="53.34" y2="27.94" width="0.4064" layer="16"/>
-<wire x1="53.34" y1="27.94" x2="50.8" y2="27.94" width="0.4064" layer="16"/>
-<wire x1="50.8" y1="5.08" x2="53.34" y2="5.08" width="0.4064" layer="16"/>
+<wire x1="55.88" y1="5.08" x2="55.88" y2="27.94" width="0.4064" layer="16"/>
+<wire x1="55.88" y1="27.94" x2="50.8" y2="27.94" width="0.4064" layer="16"/>
+<wire x1="50.8" y1="5.08" x2="55.88" y2="5.08" width="0.4064" layer="16"/>
 </signal>
 <signal name="SDA">
 <contactref element="JP3" pad="2"/>
 <contactref element="JP4" pad="5"/>
-<wire x1="50.8" y1="25.4" x2="48.26" y2="25.4" width="0.4064" layer="16"/>
-<wire x1="48.26" y1="25.4" x2="48.26" y2="5.08" width="0.4064" layer="16"/>
+<wire x1="48.26" y1="5.08" x2="48.26" y2="10.16" width="0.4064" layer="16"/>
+<wire x1="48.26" y1="10.16" x2="53.34" y2="10.16" width="0.4064" layer="16"/>
+<wire x1="53.34" y1="10.16" x2="53.34" y2="25.4" width="0.4064" layer="16"/>
+<wire x1="53.34" y1="25.4" x2="50.8" y2="25.4" width="0.4064" layer="16"/>
 </signal>
 <signal name="N$5">
